File: fitness-tracker-pcb.sch (KiCad schematic (older format))
At the start: 54 parts, among them IC1 BMD-300-A-R, IC2 BQ24230, IC3 TPS63030, IC4 LC709203F, IC5 MMBT2222ALT1G, IC6 DRV2603RUNR, IC7 W25Q128JVPIQ, Q1 BC847, U2 BAT-HLD-001, U3 APDS9960, U4 ST7735, U5 nRF52832-QFxx

Commit message: amost done arrange
Parts:
- added C21: C, Capacitor_SMD:C_0603_1608Metric, symbol Device:C
- added J1: FH33-4S-1SH_10_, FH334S1SH10, symbol FH33-4S-1SH_10_:FH33-4S-1SH_10_
Connections:
- net +2V8: no longer LS1.1 (+)
- net GND: now also U2.3
- net BAT_P: now reaches U2.1
- net BAT_P: now also C17.1, IC3.5 (VIN), LS1.1 (+), U2.2
Other:
- note removed: "ez csatlakozhatna inkább a gombelem feszültségére"
- moved on the sheet: U2
Changed lines of the file:
@@
 L BAT-HLD-001:BAT-HLD-001 U2
 U 1 1 5FD3E532
-P 4550 1600
-F 0 "U2" H 5178 1546 50  0000 L CNN
-F 1 "BAT-HLD-001" H 5178 1455 50  0000 L CNN
-F 2 "BATHLD001" H 5200 1700 50  0001 L CNN
-F 3 "" H 5200 1600 50  0001 L CNN
-F 4 "Coin Cell Battery Holders Linx CR2032 Battery Holder" H 5200 1500 50  0001 L CNN "Description"
-F 5 "4" H 5200 1400 50  0001 L CNN "Height"
-F 6 "712-BAT-HLD-001" H 5200 1300 50  0001 L CNN "Mouser Part Number"
-F 7 "https://www.mouser.co.uk/ProductDetail/Linx-Technologies/BAT-HLD-001?qs=K5ta8V%252BWhta7hbVGfm4dqA%3D%3D" H 5200 1200 50  0001 L CNN "Mouser Price/Stock"
-F 8 "Linx Technologies" H 5200 1100 50  0001 L CNN "Manufacturer_Name"
-F 9 "BAT-HLD-001" H 5200 1000 50  0001 L CNN "Manufacturer_Part_Number"
-	1    4550 1600
-	1    0    0    -1
+P 4600 800
+F 0 "U2" H 5228 746 50  0000 L CNN
+F 1 "BAT-HLD-001" H 5228 655 50  0000 L CNN
+F 2 "BATHLD001" H 5250 900 50  0001 L CNN
+F 3 "" H 5250 800 50  0001 L CNN
+F 4 "Coin Cell Battery Holders Linx CR2032 Battery Holder" H 5250 700 50  0001 L CNN "Description"
+F 5 "4" H 5250 600 50  0001 L CNN "Height"
+F 6 "712-BAT-HLD-001" H 5250 500 50  0001 L CNN "Mouser Part Number"
+F 7 "https://www.mouser.co.uk/ProductDetail/Linx-Technologies/BAT-HLD-001?qs=K5ta8V%252BWhta7hbVGfm4dqA%3D%3D" H 5250 400 50  0001 L CNN "Mouser Price/Stock"
+F 8 "Linx Technologies" H 5250 300 50  0001 L CNN "Manufacturer_Name"
+F 9 "BAT-HLD-001" H 5250 200 50  0001 L CNN "Manufacturer_Part_Number"
+	1    4600 800
+	-1   0    0    1
 $EndComp
 $Comp
@@
 $EndComp
 $Comp
-L power:+2V8 #PWR0141
-U 1 1 5FF3C9C3
-P 10000 2000
-F 0 "#PWR0141" H 10000 1850 50  0001 C CNN
-F 1 "+2V8" H 10015 2173 50  0000 C CNN
-F 2 "" H 10000 2000 50  0001 C CNN
-F 3 "" H 10000 2000 50  0001 C CNN
-	1    10000 2000
-	1    0    0    -1
-$EndComp
-Wire Notes Line
-	4400 1450 4400 2050
-Wire Notes Line
-	4400 2050 5250 2050
-Wire Notes Line
-	5250 2050 5250 1450
-Wire Notes Line
-	5250 1450 4400 1450
-$Comp
 L power:+2V8 #PWR0142
 U 1 1 5FF461A6
@@
 	1    0    0    -1
 $EndComp
-Text Notes 9400 1900 0    50   ~ 0
-ez csatlakozhatna inkább a gombelem feszültségére
+Text GLabel 4900 600  2    50   Input ~ 0
+BAT_P
+Wire Wire Line
+	4600 700  4700 700
+Wire Wire Line
+	4700 700  4700 900
+$Comp
+L power:GND #PWR0141
+U 1 1 5FE0CC73
+P 4700 900
+F 0 "#PWR0141" H 4700 650 50  0001 C CNN
+F 1 "GND" H 4705 727 50  0000 C CNN
+F 2 "" H 4700 900 50  0001 C CNN
+F 3 "" H 4700 900 50  0001 C CNN
+	1    4700 900
+	1    0    0    -1
+$EndComp
+Wire Wire Line
+	4600 800  4800 800
+Wire Wire Line
+	4800 800  4800 600
+Wire Wire Line
+	4800 600  4900 600
+Wire Wire Line
+	4600 600  4800 600
+Connection ~ 4800 600
+Text GLabel 4400 2000 0    50   Input ~ 0
+BAT_P
+Wire Wire Line
+	4400 2000 4500 2000
+Text GLabel 9900 2000 0    50   Input ~ 0
+BAT_P
+Wire Wire Line
+	9900 2000 10000 2000
+Text GLabel 9550 8350 0    50   Input ~ 0
+BUZZER
+Text GLabel 9550 8700 0    50   Input ~ 0
+GESTURE_INT
+Text GLabel 9550 8600 0    50   Input ~ 0
+GESTURE_SCL
+Text GLabel 9550 8500 0    50   Input ~ 0
+GESTURE_SDA
+Text GLabel 9550 8850 0    50   Input ~ 0
+DISPLAY_MOSI
+Text GLabel 9550 8950 0    50   Input ~ 0
+DISPLAY_SCK
+Text GLabel 9550 9050 0    50   Input ~ 0
+DISPLAY_DC
+Text GLabel 9550 9150 0    50   Input ~ 0
+DISPLAY_RESET
+Text GLabel 9550 9250 0    50   Input ~ 0
+DISPLAY_CS
+Text GLabel 9550 9350 0    50   Input ~ 0
+DISPLAY_BRIGHTNESS
+Text GLabel 9550 9500 0    50   Input ~ 0
+IMU_CS
+Text GLabel 9550 9700 0    50   Input ~ 0
+IMU_MOSI
+Text GLabel 9550 9600 0    50   Input ~ 0
+IMU_SCK
+Text GLabel 9550 9800 0    50   Input ~ 0
+IMU_MISO
+Text GLabel 9550 9900 0    50   Input ~ 0
+IMU_INT1
+Text GLabel 9550 10000 0    50   Input ~ 0
+IMU_INT2
+$Comp
+L FH33-4S-1SH_10_:FH33-4S-1SH_10_ J1
+U 1 1 5FE87160
+P 1550 4600
+F 0 "J1" H 2000 4865 50  0000 C CNN
+F 1 "FH33-4S-1SH_10_" H 2000 4774 50  0000 C CNN
+F 2 "FH334S1SH10" H 2300 4700 50  0001 L CNN
+F 3 "https://componentsearchengine.com/Datasheets/1/FH33-4S-1SH(10).pdf" H 2300 4600 50  0001 L CNN
+F 4 "HIROSE(HRS) - FH33-4S-1SH(10) - CONNECTOR, FFC/FPC, RCPT, 4POS, 1ROW" H 2300 4500 50  0001 L CNN "Description"
+F 5 "1.3" H 2300 4400 50  0001 L CNN "Height"
+F 6 "798-FH334S1SH10" H 2300 4300 50  0001 L CNN "Mouser Part Number"
+F 7 "https://www.mouser.co.uk/ProductDetail/Hirose-Connector/FH33-4S-1SH10?qs=vnk2wBG9e15DLXmQ8%2FrpIg%3D%3D" H 2300 4200 50  0001 L CNN "Mouser Price/Stock"
+F 8 "Hirose" H 2300 4100 50  0001 L CNN "Manufacturer_Name"
+F 9 "FH33-4S-1SH(10)" H 2300 4000 50  0001 L CNN "Manufacturer_Part_Number"
+	1    1550 4600
+	1    0    0    -1
+$EndComp
+$Comp
+L Device:C C21
+U 1 1 5FF9FBEE
+P 8450 8650
+F 0 "C21" H 8565 8696 50  0000 L CNN
+F 1 "C" H 8565 8605 50  0000 L CNN
+F 2 "Capacitor_SMD:C_0603_1608Metric" H 8488 8500 50  0001 C CNN
+F 3 "~" H 8450 8650 50  0001 C CNN
+	1    8450 8650
+	1    0    0    -1
+$EndComp
 $EndSCHEMATC

Commit message: before remove unnecessary parts
Connections:
- net +2V8: now also C21.1
- net BUZZER: now also IC1.31 (P0.13)
- net DISPLAY_BRIGHTNESS: now also IC1.40 (P0.22)
- net DISPLAY_CS: now also IC1.36 (P0.18)
- net DISPLAY_DC: now also IC1.26 (P0.10)
- net DISPLAY_MOSI: now also IC1.28 (P0.12)
- net DISPLAY_RESET: now also IC1.38 (P0.20)
- net DISPLAY_SCK: now also IC1.34 (P0.16)
- net GESTURE_INT: now also IC1.24 (P0.08)
- net GESTURE_SCL: now also IC1.22 (P0.06)
- net GESTURE_SDA: now also IC1.23 (P0.07)
- net GND: now also C21.2
- net IMU_CS: now also IC1.10 (P0.29)
- net IMU_INT1: now also IC1.6 (P0.25)
- net IMU_INT2: now also IC1.11 (P0.30)
- net IMU_MISO: now also IC1.7 (P0.26)
- net IMU_MOSI: now also IC1.8 (P0.27)
- net IMU_SCK: now also IC1.9 (P0.28)
Other:
- moved on the sheet: ANT1, C1, C15, C16, C2, C21, C3, C4, C5, C6, C7, C8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

Commit message: almost done 4 layer pcb
Parts:
- removed ANT1: 2450AT18B100E, ANTC3216X140N, symbol 2450AT18B100E:2450AT18B100E
- removed C1: 1.0uF, Capacitor_SMD:C_0603_1608Metric, symbol Device:C
- removed C15: 1uF, symbol Device:C
- removed C16: 0.1uF, symbol Device:C
- removed C2: 0.8pF, Capacitor_SMD:C_0402_1005Metric, symbol Device:C
- removed C3: 2.7pF, Capacitor_SMD:C_0402_1005Metric, symbol Device:C
- removed C4: 4.7uF, Capacitor_SMD:C_0603_1608Metric, symbol Device:C
- removed C5, C6, C7: 100nF, Capacitor_SMD:C_0402_1005Metric, symbol Device:C
- removed C8, C9: 100pF, Capacitor_SMD:C_0402_1005Metric, symbol Device:C
- removed IC2: BQ24230, BQ24230RGTR:QFN50P300X300X100-17N-D, symbol BQ24230RGTR:BQ24230
- removed IC4: LC709203F, LC709203FQH-01TWG:SON65P400X300X80-9N, symbol LC709203F:LC709203F
- removed IC6: DRV2603RUNR, DRV2603RUNR:QFN50P200X200X80-10N-D, symbol DRV2603RUNR:DRV2603RUNR
- removed IC7: W25Q128JVPIQ, SON127P800X600X80-9N-D, symbol W25Q128JVPIQ:W25Q128JVPIQ
- removed L1: LBMF1608T100K, INDC1608X100N, symbol LBMF1608T100K:LBMF1608T100K
- removed L2: LQP15MN2N7B02D, LQP15MN10NG02D, symbol LQP15MN2N7B02D:LQP15MN2N7B02D
- removed L3: HK100515NJ-T, INDC1005X55N, symbol HK100515NJ-T:HK100515NJ-T
- removed L4: LQP15MN3N9B02D, LQP15MN10NG02D, symbol LQP15MN3N9B02D:LQP15MN3N9B02D
- removed L5: LQP15MN1N8B02D, LQP15MN10NG02D, symbol LQP15MN1N8B02D:LQP15MN1N8B02D
- removed R10, R5, R9: 10k, symbol Device:R
- removed U5: nRF52832-QFxx, Package_DFN_QFN:QFN-48-1EP_6x6mm_P0.4mm_EP4.6x4.6mm, symbol MCU_Nordic:nRF52832-QFxx
