File: fitness-tracker-pcb.kicad_pcb (KiCad board)
At the start: 2 copper layers, 32 x 20 mm, 49 parts, among them IC1 BMD-300-A-R, IC2 BQ24230, IC3 TPS63030, IC4 LC709203F, IC5 MMBT2222ALT1G, IC6 DRV2603RUNR, IC7 W25Q128JVPIQ, Q1 BC847, U2 BAT-HLD-001, U3 APDS9960, U4 ST7735, U5 nRF52832-QFxx

Commit message: amost done arrange
Parts:
- added C21: C, Capacitor_SMD:C_0603_1608Metric, F.Cu at (51.2, 45.1)
- added J1: FH33-4S-1SH_10_, FH33-4S-1SH_10_:FH334S1SH10, B.Cu at (59.9, 39.6)
- moved C20 10.6 mm to (36.2, 43.0)
- moved IC5 9.55 mm to (36.5, 32.6), turned to 180 degrees
- moved R2 7.63 mm to (41.4, 31.5), turned to 180 degrees
- moved R3 7.12 mm to (36.2, 35.7), turned to 0 degrees
- moved C17 6.82 mm to (36.2, 49.0), turned to 0 degrees
- moved C18 5.29 mm to (40.2, 46.0), turned to 90 degrees
- moved R1 4.21 mm to (46.4, 31.5), turned to 180 degrees
- moved R7 3.88 mm to (52.2, 48.1), turned to 270 degrees
- moved R12 2.39 mm to (36.3, 40.5), turned to 270 degrees
- moved R4 2.26 mm to (42.6, 47.0)
- moved C13 2.21 mm to (42.6, 49.0), turned to 180 degrees
- moved C14 1.95 mm to (42.6, 45.1), turned to 180 degrees
- moved R13 1.82 mm to (38.2, 40.5), turned to 90 degrees
- moved C19 1.12 mm to (48.0, 34.3), turned to 180 degrees
- moved C10 0.96 mm to (48.0, 42.0)
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Connections:
- C17 pad 1: Net-(C17-Pad1) -> BAT_P
- IC3 pad 5: Net-(C17-Pad1) -> BAT_P
- LS1 pad 1: +2V8 -> BAT_P
- U2 pad 1: Net-(U2-Pad1) -> BAT_P
- U2 pad 2: Net-(U2-Pad2) -> BAT_P
- U2 pad 3: Net-(U2-Pad3) -> GND

Commit message: add 2 inner layer
Routing:
- added copper zone on PWR, net +2V8
- added copper zone on GND, net GND
Other:
- copper layers 2 -> 4

Commit message: add some wiring
Parts:
- turned LS1 to 0 degrees
Routing:
- net GND: track 0.00 -> 13.0 mm, vias 0 -> 2
- net +2V8: track 0.00 -> 10.6 mm, vias 0 -> 1
- net BAT_P: track 0.00 -> 4.82 mm, vias 0 -> 1
- net Net-(IC3-Pad4): track 0.00 -> 3.99 mm
- net Net-(IC3-Pad2): track 0.00 -> 3.99 mm
- added copper zone on B.Cu, net BAT_P
- added copper zone on F.Cu, net GND
Other:
- net class Plus added: clearance 0.2, trace_width 0.625, via_dia 0.8, via_drill 0.4

Commit message: before remove unnecessary parts
Parts:
- moved R11 6.58 mm to (60.6, 47.0)
- moved C12 5.85 mm to (41.8, 48.2), turned to 90 degrees
- moved R4 4.49 mm to (46.0, 44.1), turned to 0 degrees
- moved R7 3.90 mm to (49.2, 45.6), turned to 180 degrees
- moved R12 2.68 mm to (36.3, 37.8), turned to 0 degrees
- moved R6 1.57 mm to (48.1, 48.2), turned to 90 degrees
- moved C13 1.53 mm to (43.9, 48.2), turned to 90 degrees
- moved C21 1.41 mm to (52.6, 45.6)
- moved R8 1.38 mm to (50.2, 48.2), turned to 90 degrees
- moved R13 1.16 mm to (37.1, 40.6), turned to 270 degrees
- moved LS1 0.60 mm to (57.4, 47.0)
- moved Q1 0.60 mm to (57.4, 47.0), turned to 180 degrees
- moved C14 0.55 mm to (42.9, 45.6)
- moved AC1 0.25 mm to (48.2, 39.3)
- moved C10 0.25 mm to (48.2, 42.0)
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Connections:
- C21 pad 1: Net-(C21-Pad1) -> +2V8
- C21 pad 2: Net-(C21-Pad2) -> GND
- IC1 pad 10: Net-(IC1-Pad10) -> IMU_CS
- IC1 pad 11: Net-(IC1-Pad11) -> IMU_INT2
- IC1 pad 22: Net-(IC1-Pad22) -> GESTURE_SCL
- IC1 pad 23: Net-(IC1-Pad23) -> GESTURE_SDA
- IC1 pad 24: Net-(IC1-Pad24) -> GESTURE_INT
- IC1 pad 26: Net-(IC1-Pad26) -> DISPLAY_DC
- IC1 pad 28: Net-(IC1-Pad28) -> DISPLAY_MOSI
- IC1 pad 31: Net-(IC1-Pad31) -> BUZZER
- IC1 pad 34: Net-(IC1-Pad34) -> DISPLAY_SCK
- IC1 pad 36: Net-(IC1-Pad36) -> DISPLAY_CS
- IC1 pad 38: Net-(IC1-Pad38) -> DISPLAY_RESET
- IC1 pad 40: Net-(IC1-Pad40) -> DISPLAY_BRIGHTNESS
- IC1 pad 6: Net-(IC1-Pad6) -> IMU_INT1
- IC1 pad 7: Net-(IC1-Pad7) -> IMU_MISO
- IC1 pad 8: Net-(IC1-Pad8) -> IMU_MOSI
- IC1 pad 9: Net-(IC1-Pad9) -> IMU_SCK
- LS1 pad 1: BAT_P -> DISPLAY_DC
- U2 pad 1: BAT_P -> DISPLAY_DC
Routing:
- net GND: track 13.0 -> 49.2 mm, vias 2 -> 10
- net +2V8: track 10.6 -> 40.0 mm, vias 1 -> 6
- net DISPLAY_DC: track 0.00 -> 26.1 mm, vias 0 -> 2
- net DISPLAY_RESET: track 0.00 -> 22.5 mm, vias 0 -> 2
- net DISPLAY_CS: track 0.00 -> 20.2 mm, vias 0 -> 2
- net DISPLAY_MOSI: track 0.00 -> 15.4 mm, vias 0 -> 2
- net DISPLAY_SCK: track 0.00 -> 15.1 mm, vias 0 -> 2
- net GESTURE_SCL: track 0.00 -> 14.2 mm
- net GESTURE_INT: track 0.00 -> 13.4 mm
- net GESTURE_SDA: track 0.00 -> 11.7 mm
- net Net-(IC3-Pad10): track 0.00 -> 7.68 mm
- net IMU_INT1: track 0.00 -> 4.66 mm
- net BUZZER: track 0.00 -> 4.20 mm
- net Net-(IC5-Pad1): track 0.00 -> 3.94 mm
- net Net-(C14-Pad1): track 0.00 -> 3.87 mm
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Other:
- net class IMU added: clearance 0.2, trace_width 0.2, via_dia 0.8, via_drill 0.4

Commit message: almost done 4 layer pcb
Parts:
- removed ANT1: 2450AT18B100E, 2450AT18B100E:ANTC3216X140N
- removed C1: 1.0uF, Capacitor_SMD:C_0603_1608Metric
- removed C2: 0.8pF, Capacitor_SMD:C_0402_1005Metric
- removed C3: 2.7pF, Capacitor_SMD:C_0402_1005Metric
- removed C4: 4.7uF, Capacitor_SMD:C_0603_1608Metric
- removed C5, C6, C7: 100nF, Capacitor_SMD:C_0402_1005Metric
- removed C8, C9: 100pF, Capacitor_SMD:C_0402_1005Metric
- removed IC2: BQ24230, BQ24230RGTR:QFN50P300X300X100-17N-D
- removed IC4: LC709203F, LC709203FQH-01TWG:SON65P400X300X80-9N
- removed IC6: DRV2603RUNR, DRV2603RUNR:QFN50P200X200X80-10N-D
- removed IC7: W25Q128JVPIQ, W25Q128JVPIQ:SON127P800X600X80-9N-D
- removed L1: LBMF1608T100K, LBMF1608T100K:INDC1608X100N
- removed L2: LQP15MN2N7B02D, LQP15MN1N8B02D:LQP15MN10NG02D
- removed L3: HK100515NJ-T, HK100515NJ-T:INDC1005X55N
- removed L4: LQP15MN3N9B02D, LQP15MN1N8B02D:LQP15MN10NG02D
- removed L5: LQP15MN1N8B02D, LQP15MN1N8B02D:LQP15MN10NG02D
- removed U5: nRF52832-QFxx, Package_DFN_QFN:QFN-48-1EP_6x6mm_P0.4mm_EP4.6x4.6mm

Commit message: done? drv good!
Connections:
- LS1 pad 1: DISPLAY_DC -> BAT_P
- U2 pad 1: DISPLAY_DC -> BAT_P
Routing:
- net DISPLAY_BRIGHTNESS: track 3.35 -> 20.4 mm, vias 0 -> 2
- net GND: track 49.2 -> 63.5 mm, vias 10 -> 17
- net DISPLAY_DC: track 26.1 -> 18.9 mm
- net Net-(R3-Pad2): track 0.00 -> 6.85 mm
- net +2V8: track 40.0 -> 46.4 mm
- net BAT_P: track 4.82 -> 10.9 mm
